File: charger.kicad_pcb (KiCad board)
At the start: 2 copper layers, 520 x 166.3 mm, 41 parts, among them J1 1714971, U1 TP4056, U10 TP4056, U11 TP4056, U12 TP4056, U13 TP4056, U14 TP4056, U15 TP4056, U16 TP4056, U17 TP4056, U18 TP4056, U19 TP4056, U2 TP4056, U20 TP4056, U3 TP4056, U4 TP4056, U5 TP4056, U6 TP4056, U7 TP4056, U8 TP4056, U9 TP4056

Commit message: added mounting holes
Parts:
- added H1: MountingHole, MountingHole:MountingHole_2.7mm_M2.5, F.Cu at (68.9, 117.9)
- added H10: MountingHole, MountingHole:MountingHole_2.7mm_M2.5, F.Cu at (518.9, 117.9)
- added H11: MountingHole, MountingHole:MountingHole_2.7mm_M2.5, F.Cu at (68.9, 195.9)
- added H12: MountingHole, MountingHole:MountingHole_2.7mm_M2.5, F.Cu at (118.9, 195.9)
- added H13: MountingHole, MountingHole:MountingHole_2.7mm_M2.5, F.Cu at (168.9, 195.9)
- added H14: MountingHole, MountingHole:MountingHole_2.7mm_M2.5, F.Cu at (218.9, 195.9)
- added H15: MountingHole, MountingHole:MountingHole_2.7mm_M2.5, F.Cu at (268.9, 195.9)
- added H16: MountingHole, MountingHole:MountingHole_2.7mm_M2.5, F.Cu at (318.9, 195.9)
- added H17: MountingHole, MountingHole:MountingHole_2.7mm_M2.5, F.Cu at (368.9, 195.9)
- added H18: MountingHole, MountingHole:MountingHole_2.7mm_M2.5, F.Cu at (418.9, 195.9)
- added H19: MountingHole, MountingHole:MountingHole_2.7mm_M2.5, F.Cu at (468.9, 195.9)
- added H2: MountingHole, MountingHole:MountingHole_2.7mm_M2.5, F.Cu at (118.9, 117.9)
- added H20: MountingHole, MountingHole:MountingHole_2.7mm_M2.5, F.Cu at (518.9, 195.9)
- added H3: MountingHole, MountingHole:MountingHole_2.7mm_M2.5, F.Cu at (168.9, 117.9)
- added H4: MountingHole, MountingHole:MountingHole_2.7mm_M2.5, F.Cu at (218.9, 117.9)
- added H5: MountingHole, MountingHole:MountingHole_2.7mm_M2.5, F.Cu at (268.9, 117.9)
- added H6: MountingHole, MountingHole:MountingHole_2.7mm_M2.5, F.Cu at (318.9, 117.9)
- added H7: MountingHole, MountingHole:MountingHole_2.7mm_M2.5, F.Cu at (368.9, 117.9)
- added H8: MountingHole, MountingHole:MountingHole_2.7mm_M2.5, F.Cu at (418.9, 117.9)
- added H9: MountingHole, MountingHole:MountingHole_2.7mm_M2.5, F.Cu at (468.9, 117.9)
- moved BT10 301.1 mm to (518.9, 186.7)
- moved U10 301.1 mm to (538.9, 144.7)
- moved BT12 278.5 mm to (118.9, 264.7)
- moved BT13 278.5 mm to (168.9, 264.7)
- moved U12 278.5 mm to (138.9, 222.7)
- moved U13 278.5 mm to (188.9, 222.7)
- moved BT6 251.6 mm to (318.9, 186.7)
- moved BT7 251.6 mm to (368.9, 186.7)
- moved BT8 251.6 mm to (418.9, 186.7)
- moved U6 251.6 mm to (338.9, 144.7)
- moved U7 251.6 mm to (388.9, 144.7)
- moved U8 251.6 mm to (438.9, 144.7)
- moved BT9 229.6 mm to (468.9, 186.7)
- moved U9 229.6 mm to (488.9, 144.7)
- moved BT16 217.6 mm to (318.9, 264.7)
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Routing:
- net /GND: track 1448.6 -> 1579.4 mm
- net /5V: track 1465.1 -> 1569.7 mm
- net Net-(BT15-Pad1): track 68.9 -> 67.6 mm
- net Net-(BT13-Pad1): track 67.4 -> 68.5 mm
- net Net-(BT9-Pad1): track 67.9 -> 67.1 mm
- net Net-(BT16-Pad1): track 67.1 -> 67.9 mm
- net Net-(BT6-Pad1): track 68.8 -> 67.9 mm
- net Net-(BT12-Pad1): track 67.9 -> 68.8 mm
- net Net-(BT10-Pad1): track 67.6 -> 68.3 mm
- net Net-(BT7-Pad1): track 68.5 -> 67.9 mm
- net Net-(BT14-Pad1): track 67.9 -> 67.4 mm
Other:
- board size 520 x 166.3 mm -> 530 x 170 mm

Commit message: added filed zones
Parts:
- renumbered BT15 to BT10, BT7 to BT12, BT8 to BT13, BT16 to BT14, BT17 to BT15, BT9 to BT16, BT18 to BT17, BT10 to BT18, BT12 to BT6, BT13 to BT7, BT14 to BT8, BT6 to BT9, H11 to H10, H12 to H11, H13 to H12, H14 to H13, H15 to H14, H16 to H15, H17 to H16, H18 to H17, H19 to H18, H20 to H19, H9 to H20, H10 to H9, U15 to U10, U7 to U12, U8 to U13, U16 to U14, U17 to U15, U9 to U16, U18 to U17, U10 to U18, U12 to U6, U13 to U7, U14 to U8, U6 to U9
Connections:
- BT1 pad 2: Net-(BT1-Pad2) -> /GND
- BT10 pad 2: Net-(BT10-Pad2) -> /GND
- BT11 pad 2: Net-(BT11-Pad2) -> /GND
- BT12 pad 2: Net-(BT12-Pad2) -> /GND
- BT13 pad 2: Net-(BT13-Pad2) -> /GND
- BT14 pad 2: Net-(BT14-Pad2) -> /GND
- BT15 pad 2: Net-(BT15-Pad2) -> /GND
- BT16 pad 2: Net-(BT16-Pad2) -> /GND
- BT17 pad 2: Net-(BT17-Pad2) -> /GND
- BT18 pad 2: Net-(BT18-Pad2) -> /GND
- BT19 pad 2: Net-(BT19-Pad2) -> /GND
- BT2 pad 2: Net-(BT2-Pad2) -> /GND
- BT20 pad 2: Net-(BT20-Pad2) -> /GND
- BT3 pad 2: Net-(BT3-Pad2) -> /GND
- BT4 pad 2: Net-(BT4-Pad2) -> /GND
- BT5 pad 2: Net-(BT5-Pad2) -> /GND
- BT6 pad 2: Net-(BT6-Pad2) -> /GND
- BT7 pad 2: Net-(BT7-Pad2) -> /GND
- BT8 pad 2: Net-(BT8-Pad2) -> /GND
- BT9 pad 2: Net-(BT9-Pad2) -> /GND
- U1 pad 4: Net-(BT1-Pad2) -> /GND
- U10 pad 4: Net-(BT10-Pad2) -> /GND
- U11 pad 4: Net-(BT11-Pad2) -> /GND
- U12 pad 4: Net-(BT12-Pad2) -> /GND
- U13 pad 4: Net-(BT13-Pad2) -> /GND
- U14 pad 4: Net-(BT14-Pad2) -> /GND
- U15 pad 4: Net-(BT15-Pad2) -> /GND
- U16 pad 4: Net-(BT16-Pad2) -> /GND
- U17 pad 4: Net-(BT17-Pad2) -> /GND
- U18 pad 4: Net-(BT18-Pad2) -> /GND
- U19 pad 4: Net-(BT19-Pad2) -> /GND
- U2 pad 4: Net-(BT2-Pad2) -> /GND
- U20 pad 4: Net-(BT20-Pad2) -> /GND
- U3 pad 4: Net-(BT3-Pad2) -> /GND
- U4 pad 4: Net-(BT4-Pad2) -> /GND
- U5 pad 4: Net-(BT5-Pad2) -> /GND
- U6 pad 4: Net-(BT6-Pad2) -> /GND
- U7 pad 4: Net-(BT7-Pad2) -> /GND
- U8 pad 4: Net-(BT8-Pad2) -> /GND
- U9 pad 4: Net-(BT9-Pad2) -> /GND
Routing:
- net /GND: track 1579.4 -> 1.79 mm
- net /5V: track 1569.7 -> 1.79 mm
- net Net-(BT1-Pad2): track 64.0 -> 0.00 mm
- net Net-(BT9-Pad2): track 64.0 -> 0.00 mm
- net Net-(BT4-Pad2): track 64.0 -> 0.00 mm
- net Net-(BT3-Pad2): track 64.0 -> 0.00 mm
- net Net-(BT2-Pad2): track 64.0 -> 0.00 mm
- net Net-(BT16-Pad2): track 64.0 -> 0.00 mm
- net Net-(BT13-Pad2): track 64.0 -> 0.00 mm
- net Net-(BT12-Pad2): track 64.0 -> 0.00 mm
- net Net-(BT5-Pad2): track 64.0 -> 0.00 mm
- net Net-(BT18-Pad2): track 64.0 -> 0.00 mm
- net Net-(BT11-Pad2): track 64.0 -> 0.00 mm
- net Net-(BT8-Pad2): track 64.0 -> 0.00 mm
- net Net-(BT7-Pad2): track 64.0 -> 0.00 mm
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- added copper zone on F.Cu, net /5V
- added copper zone on B.Cu, net /GND
Other:
- board text added: "IRIDIA"
- board text added: "e-puck battery charger V1.0"
